Commit message: Blunder Update

File: description/imu.xacro (robot description, xacro)
@@ -3,5 +3,5 @@
     <joint name="imu_joint" type="fixed">
         <parent link="base_link"/>
-        <child link="imu_link"/>
+        <child link="imu"/>
         <origin xyz="0 0 0.115" rpy="0 0 0"/>
     </joint>

Commit message: Update [IMU-ODOM]

File: description/imu.xacro (robot description, xacro)
@@ -2,5 +2,5 @@
 <robot xmlns:xacro="http://www.ros.org/wiki/xacro">
     <joint name="imu_joint" type="fixed">
-        <parent link="base_link"/>
+        <parent link="chassis"/>
         <child link="imu"/>
         <origin xyz="0 0 0.115" rpy="0 0 0"/>

File: description/lidar.xacro (robot description, xacro)
@@ -1,10 +1,4 @@
 <?xml version="1.0"?>
 <robot xmlns:xacro="http://www.ros.org/wiki/xacro">
-    <!-- <joint name="base_footprint_joint" type="fixed">
-        <parent link="base_link"/>
-        <child link="base_footprint"/>
-        <origin xyz="0.0 0.0 0.0" rpy="0.0 0.0 0.0"/>
-    </joint>
-    <link name="base_footprint"></link> -->
     <link name="laser">
         <visual>
@@ -37,7 +31,7 @@
                 <scan>
                     <horizontal>
-                        <samples>180</samples>
-                        <min_angle>-1.57</min_angle>
-                        <max_angle>1.57</max_angle>
+                        <samples>360</samples>
+                        <min_angle>-3.14</min_angle>
+                        <max_angle>3.14</max_angle>
                     </horizontal>
                 </scan>

File: description/robot_core.xacro (robot description, xacro)
@@ -54,12 +54,12 @@
     </link>
     <!-- BASE FOOTPRINT JOINT -->
-    <!-- <joint name="base_footprint_joint" type="fixed">
+    <joint name="base_footprint_joint" type="fixed">
         <parent link="base_link"/>
         <child link="base_footprint"/>
         <origin xyz="0 0 0" rpy="0 0 0"/>
-    </joint> -->
+    </joint>
     <!-- BASE FOOTPRINT LINK -->
-    <!-- <link name="base_footprint">
-    </link> -->
+    <link name="base_footprint">
+    </link>
     <!-- ================================================================================== -->
     <!-- CHASSIS JOINT -->
@@ -67,5 +67,5 @@
         <parent link="base_link"/>
         <child link="chassis"/>
-        <origin xyz="0 0 ${-wheel_offset_z}"/>
+        <origin xyz="0 0 ${-wheel_offset_z}" rpy="0 0 0"/>
     </joint>
     <!-- CHASSIS LINK -->
@@ -98,5 +98,5 @@
     <!-- LEFT WHEEL JOINT -->
     <joint name="left_wheel_joint" type="continuous">
-        <parent link="base_link"/>
+        <parent link="chassis"/>
         <child link="left_wheel"/>
         <origin xyz="-0.01 ${wheel_offset_y} 0" rpy="-${pi/2} 0 0" />
@@ -130,5 +130,5 @@
     <!-- RIGHT WHEEL JOINT -->
     <joint name="right_wheel_joint" type="continuous">
-        <parent link="base_link"/>
+        <parent link="chassis"/>
         <child link="right_wheel"/>
         <origin xyz="-0.01 ${-wheel_offset_y} 0" rpy="${pi/2} 0 0"/>
@@ -163,5 +163,5 @@
     <!-- REAR CASTER WHEEL JOINT -->
     <joint name="rear_caster_wheel_joint" type="fixed">
-        <parent link="base_link"/>
+        <parent link="chassis"/>
         <child link="rear_caster_wheel"/>
         <origin xyz="${-caster_wheel_offset_x} 0 ${caster_wheel_offset_z}"/>
@@ -227,5 +227,5 @@
     <!-- RIGHT CASTER WHEEL 2 -->
     <joint name="right_caster_wheel_joint" type="fixed">
-        <parent link="base_link"/>
+        <parent link="chassis"/>
         <child link="right_caster_wheel"/>
         <origin xyz="0.15 ${-caster_wheel_offset_y} ${caster_wheel_offset_z}"/>
