Commit message: Reverting Changes, Deleted my_controller, ros2_control xacro files

File: description/lidar.xacro (robot description, xacro)
@@ -1,10 +1,10 @@
 <?xml version="1.0"?>
 <robot xmlns:xacro="http://www.ros.org/wiki/xacro">
-    <link name="base_footprint"></link>
-    <joint name="base_footprint_joint" type="fixed">
+    <!-- <joint name="base_footprint_joint" type="fixed">
         <parent link="base_link"/>
         <child link="base_footprint"/>
         <origin xyz="0.0 0.0 0.0" rpy="0.0 0.0 0.0"/>
     </joint>
+    <link name="base_footprint"></link> -->
     <link name="laser">
         <visual>

File: description/robot.urdf.xacro (robot description, xacro)
@@ -1,18 +1,6 @@
 <?xml version="1.0"?>
 <robot xmlns:xacro="http://www.ros.org/wiki/xacro"  name="robot">
-     <!-- Arguments -->
-    <xacro:arg name="use_ros2_control" default="true" />
-    <xacro:arg name="use_sim_time" default="false" />
-    <!-- Include the ROS URDF -->
-    <xacro:include filename="robot_core.xacro" />
-    <xacro:if value="$(arg use_ros2_control)">
-        <!-- ROS2 Control -->
-        <xacro:include filename="ros2_control.xacro" />
-    </xacro:if>
-    <xacro:unless value="$(arg  use_ros2_control)">
-        <!-- Legacy ros control -->
-        <xacro:include filename="gazebo_control.xacro" />
-    </xacro:unless>
-    <!-- Lidar  Sensor -->
+    <xacro:include filename="robot_core.xacro"/>
+    <xacro:include filename="gazebo_control.xacro"/>
     <xacro:include filename="lidar.xacro"/>
 </robot>

File: description/robot_core.xacro (robot description, xacro)
@@ -13,5 +13,5 @@
     <xacro:property name="wheel_offset_z" value="0.005"/>
     <!-- WHEELS PARAMETERS -->
-    <xacro:property name="wheel_radius" value="0.1"/>
+    <xacro:property name="wheel_radius" value="0.05"/>
     <xacro:property name="wheel_thickness" value="0.026"/>
     <xacro:property name="wheel_mass" value="0.05"/>
@@ -54,12 +54,12 @@
     </link>
     <!-- BASE FOOTPRINT JOINT -->
-    <joint name="base_footprint_joint" type="fixed">
+    <!-- <joint name="base_footprint_joint" type="fixed">
         <parent link="base_link"/>
         <child link="base_footprint"/>
         <origin xyz="0 0 0" rpy="0 0 0"/>
-    </joint>
+    </joint> -->
     <!-- BASE FOOTPRINT LINK -->
-    <link name="base_footprint">
-    </link>
+    <!-- <link name="base_footprint">
+    </link> -->
     <!-- ================================================================================== -->
     <!-- CHASSIS JOINT -->

Commit message: hardware

File: description/lidar.xacro (robot description, xacro)
@@ -1,10 +1,4 @@
 <?xml version="1.0"?>
 <robot xmlns:xacro="http://www.ros.org/wiki/xacro">
-    <!-- <joint name="base_footprint_joint" type="fixed">
-        <parent link="base_link"/>
-        <child link="base_footprint"/>
-        <origin xyz="0.0 0.0 0.0" rpy="0.0 0.0 0.0"/>
-    </joint>
-    <link name="base_footprint"></link> -->
     <link name="laser">
         <visual>

File: description/robot_core.xacro (robot description, xacro)
@@ -53,4 +53,10 @@
     <link name="base_link">
     </link>
+    <link name="imu_link"></link>
+    <joint name="imu_joint" type="fixed">
+        <parent link="chassis"/>
+        <child link="imu_link"/>
+        <origin xyz="0.0 0.0 0.0" rpy="0.0 0.0 0.0"/>
+    </joint>
     <!-- BASE FOOTPRINT JOINT -->
     <joint name="base_footprint_joint" type="fixed">

File: description/ros2_control.xacro (robot description, xacro)
@@ -10,5 +10,5 @@
             <param name="timeout_ms">1000</param>
             <param name="loop_rate">30</param>
-            <param name="enc_counts_per_rev">5042</param>
+            <param name="enc_counts_per_rev">752</param>
         </hardware>
         <joint name="left_wheel_joint">

Commit message: Minor Update

File: description/lidar.xacro (robot description, xacro)
@@ -26,5 +26,5 @@
         <parent link="chassis"/>
         <child link="laser"/>
-        <origin xyz="0.0 0.0 0.13" rpy="0.0 0.0 0.0"/>
+        <origin xyz="0.140 0.0 0.13" rpy="0.0 0.0 0.0"/>
     </joint>
     <gazebo reference="laser">

Commit message: updated

File: description/lidar.xacro (robot description, xacro)
@@ -20,5 +20,5 @@
         <parent link="chassis"/>
         <child link="laser"/>
-        <origin xyz="0.0 0.0 0.13" rpy="0.0 0.0 0.0"/>
+        <origin xyz="0.140 0.0 0.13" rpy="0.0 0.0 3.14"/>
     </joint>
     <gazebo reference="laser">
@@ -31,7 +31,7 @@
                 <scan>
                     <horizontal>
-                        <samples>180</samples>
-                        <min_angle>-1.57</min_angle>
-                        <max_angle>1.57</max_angle>
+                        <samples>360</samples>
+                        <min_angle>-3.14</min_angle>
+                        <max_angle>3.14</max_angle>
                     </horizontal>
                 </scan>

Commit message: added navigation

File: description/lidar.xacro (robot description, xacro)
@@ -20,5 +20,5 @@
         <parent link="chassis"/>
         <child link="laser"/>
-        <origin xyz="0.140 0.0 0.13" rpy="0.0 0.0 3.14"/>
+        <origin xyz="0.140 0.0 0.13" rpy="0.0 0.0 0"/>
     </joint>
     <gazebo reference="laser">

File: description/robot.urdf.xacro (robot description, xacro)
@@ -4,4 +4,5 @@
     <xacro:include filename="robot_core.xacro"/>
     <xacro:include filename="lidar.xacro"/>
+    <xacro:include filename="imu.xacro"/>
     <xacro:if value="$(arg use_ros2_control)">
         <xacro:include filename="ros2_control.xacro"/>

File: description/robot_core.xacro (robot description, xacro)
@@ -53,10 +53,4 @@
     <link name="base_link">
     </link>
-    <link name="imu_link"></link>
-    <joint name="imu_joint" type="fixed">
-        <parent link="chassis"/>
-        <child link="imu_link"/>
-        <origin xyz="0.0 0.0 0.0" rpy="0.0 0.0 0.0"/>
-    </joint>
     <!-- BASE FOOTPRINT JOINT -->
     <joint name="base_footprint_joint" type="fixed">

Commit message: Update Inverted URDF, Update 45 Deg TOF, Update Range to LaserScan

File: description/lidar.xacro (robot description, xacro)
@@ -20,5 +20,5 @@
         <parent link="chassis"/>
         <child link="laser"/>
-        <origin xyz="0.140 0.0 0.13" rpy="0.0 0.0 0.0"/>
+        <origin xyz="0.140 0.0 0.13" rpy="0.0 0.0 ${pi}"/>
     </joint>
     <gazebo reference="laser">

File: description/tof.xacro (robot description, xacro)
@@ -47,5 +47,5 @@
         <parent link="chassis"/>
         <child link="tof_1"/>
-        <origin xyz="0.192 0.148 0.06" rpy="0 0 0"/>
+        <origin xyz="0.192 0.148 0.06" rpy="0 0 ${pi/4}"/>
     </joint>
     <link name="tof_2">
@@ -68,5 +68,5 @@
         <parent link="chassis"/>
         <child link="tof_2"/>
-        <origin xyz="0.192 -0.148 0.06" rpy="0 0 0"/>
+        <origin xyz="0.192 -0.148 0.06" rpy="0 0 -${pi/4}"/>
     </joint>
     <gazebo reference="tof">
