Commit message: Updated [Res. Nav, Multi_Nav, Single_Nav]

File: description/tof.xacro (robot description, xacro)
@@ -47,5 +47,5 @@
         <parent link="chassis"/>
         <child link="tof_1"/>
-        <origin xyz="0.192 0.148 0.06" rpy="0 0 ${pi/4}"/>
+        <origin xyz="0.192 0.148 0.06" rpy="0 0 0.523599"/>
     </joint>
     <link name="tof_2">
@@ -68,5 +68,5 @@
         <parent link="chassis"/>
         <child link="tof_2"/>
-        <origin xyz="0.192 -0.148 0.06" rpy="0 0 -${pi/4}"/>
+        <origin xyz="0.192 -0.148 0.06" rpy="0 0 -0.523599"/>
     </joint>
     <gazebo reference="tof">
