Commit message: urdf and inertia update

File: description/robot_core.xacro (robot description, xacro)
@@ -21,4 +21,5 @@
     <xacro:property name="caster_wheel_offset_x" value="0.075"/>
     <xacro:property name="caster_wheel_offset_z" value="${wheel_offset_z - wheel_radius + castor_wheel_radius}"/>
+    <!-- ================================================================================== -->
     <!-- XACRO COLORS -->
     <material name="white">
@@ -46,5 +47,5 @@
         <color rgba="0.7 0.7 0.7 1.0"/>
     </material>
-    <!-- ========================================================= -->
+    <!-- ================================================================================== -->
     <!-- BASE FOOTPRINT -->
     <!-- BASE LINK -->
@@ -57,4 +58,5 @@
         <origin xyz="${-wheel_offset_x} 0 ${-wheel_offset_z}"/>
     </joint>
+    <!-- ================================================================================== -->
     <!-- CHASSIS LINK -->
     <link name="chassis">
@@ -75,5 +77,13 @@
         </collision>
         <!-- INERTIA -->
-    </link>
+        <xacro:inertial_cylinder mass="${chassis_mass}" length="${chassis_thickness}" radius="${chassis_radius}">
+            <origin xyz="0 0 0" rpy="0 0 0"/>
+        </xacro:inertial_cylinder>
+    </link>
+    <!-- GAZEBO CHASSIS -->
+    <gazebo refernce="chassis">
+        <material>Gazebo/Silver</material>
+    </gazebo>
+    <!-- ================================================================================== -->
     <!-- LEFT WHEEL JOINT -->
     <joint name="left_wheel_joint", type="continous">
@@ -99,5 +109,13 @@
         </collision>
         <!-- INERTIA -->
-    </link>
+        <xacro:inertial_cylinder mass="${wheel_mass}" length="${wheel_thickness}" radius="${wheel_radius}">
+            <origin xyz="0 0 0" rpy="0 0 0"/>
+        </xacro:inertial_cylinder>
+    </link>
+    <!-- GAZEBO LEFT WHEEL -->
+    <gazebo refernce="left_wheel">
+        <material>Gazebo/Blue</material>
+    </gazebo>
+    <!-- ================================================================================== -->
     <!-- RIGHT WHEEL JOINT -->
     <joint name="right_wheel_joint" type="continous">
@@ -123,5 +141,13 @@
         </collision>
         <!-- INERTIA -->
-    </link>
+        <xacro:inertial_cylinder mass="${wheel_mass}" length="${wheel_thickness}" radius="${wheel_radius}">
+            <origin xyz="0 0 0" rpy="0 0 0"/>
+        </xacro:inertial_cylinder>
+    </link>
+    <!-- GAZEBO RIGHT WHEEL -->
+    <gazebo refrence="right_wheel">
+        <material>Gazebo/Blue</material>
+    </gazebo>
+    <!-- ================================================================================== -->
     <!-- REAR CASTER WHEEL -->
     <!-- REAR CASTER WHEEL JOINT -->
@@ -147,5 +173,14 @@
         </collison>
         <!-- INERTIA -->
-    </link>
+        <xacro:inertial_sphere mass="${caster_wheel_mass}" radius="${caster_wheel_radius}">
+            <origin xyz="0 0 0" rpy="0 0 0"/>
+        </xacro:inertial_sphere>
+    </link>
+    <!-- GAZEBO REAR CASTER WHEEL -->
+     <gazebo reference="rear_caster_wheel">
+        <material>Gazebo/Black</material>
+        <mu1 value="0.001"/>
+        <mu2 value="0.001"/>
+    </gazebo>
     <!-- LEFT CASTER WHEEL  -->
     <joint name="left_caster_wheel_joint" type="fixed">
@@ -170,5 +205,14 @@
         </collison>
         <!-- INERTIA -->
-    </link>
+        <xacro:inertial_sphere mass="${caster_wheel_mass}" radius="${caster_wheel_radius}">
+            <origin xyz="0 0 0" rpy="0 0 0"/>
+        </xacro:inertial_sphere>
+    </link>
+    <!-- GAZEBO LEFT CASTER WHEEL -->
+     <gazebo reference="left_caster_wheel">
+        <material>Gazebo/Black</material>
+        <mu1 value="0.001"/>
+        <mu2 value="0.001"/>
+    </gazebo>
     <!-- RIGHT CASTER WHEEL 2 -->
     <joint name="right_caster_wheel_joint" type="fixed">
@@ -193,4 +237,13 @@
         </collison>
         <!-- INERTIA -->
-    </link>
+        <xacro:inertial_sphere mass="${caster_wheel_mass}" radius="${caster_wheel_radius}">
+            <origin xyz="0 0 0" rpy="0 0 0"/>
+        </xacro:inertial_sphere>
+    </link>
+    <!-- GAZEBO RIGHT CASTER WHEEL -->
+     <gazebo reference="right_caster_wheel">
+        <material>Gazebo/Black</material>
+        <mu1 value="0.001"/>
+        <mu2 value="0.001"/>
+    </gazebo>
 </robot>

Commit message: Update

File: description/robot_core.xacro (robot description, xacro)
@@ -1,5 +1,5 @@
 <?xml version="1.0"?>
 <robot xmlns:xacro="http://www.ros.org/wiki/xacro"  name="robot">
-    <xacro:include filename="intertial_macros.xacro"/>
+    <xacro:include filename="inertial_macros.xacro"/>
     <!-- PARAMETERS -->
     <!-- CHASSIS PARAMETERS -->
@@ -20,5 +20,5 @@
     <!-- CASTER WHEEL OFFSET PARAMTERS -->
     <xacro:property name="caster_wheel_offset_x" value="0.075"/>
-    <xacro:property name="caster_wheel_offset_z" value="${wheel_offset_z - wheel_radius + castor_wheel_radius}"/>
+    <xacro:property name="caster_wheel_offset_z" value="${wheel_offset_z - wheel_radius + caster_wheel_radius}"/>
     <!-- ================================================================================== -->
     <!-- XACRO COLORS -->
@@ -37,5 +37,5 @@
     <material name="blue">
         <color rgba="0.2 0.2 1 1"/>
-    <material>
+    </material>
     <material name="black">
         <color rgba="0 0 0 1"/>
@@ -63,5 +63,5 @@
         <!-- VISUAL -->
         <visual>
-            <origin xyz="${chassis_radius/2} 0 ${chassis_height/2}"/>
+            <origin xyz="${chassis_radius/2} 0 ${chassis_thickness}"/>
             <geometry>
                 <cylinder radius="${chassis_radius}" length="${chassis_thickness}"/>
@@ -71,5 +71,5 @@
         <!-- COLLISION -->
         <collision>
-            <origin xyz="${chassis_radius/2} 0 ${chassis_height/2}"/>
+            <origin xyz="${chassis_radius/2} 0 ${chassis_thickness}"/>
             <geometry>
                 <cylinder radius="${chassis_radius}" length="${chassis_thickness}"/>
@@ -87,5 +87,5 @@
     <!-- ================================================================================== -->
     <!-- LEFT WHEEL JOINT -->
-    <joint name="left_wheel_joint", type="continous">
+    <joint name="left_wheel_joint" type="continous">
         <parent link="base_link"/>
         <child link="left_wheel"/>
@@ -171,5 +171,5 @@
                 <sphere radius="${caster_wheel_radius}"/>
             </geometry>
-        </collison>
+        </collision>
         <!-- INERTIA -->
         <xacro:inertial_sphere mass="${caster_wheel_mass}" radius="${caster_wheel_radius}">
@@ -178,5 +178,5 @@
     </link>
     <!-- GAZEBO REAR CASTER WHEEL -->
-     <gazebo reference="rear_caster_wheel">
+    <gazebo reference="rear_caster_wheel">
         <material>Gazebo/Black</material>
         <mu1 value="0.001"/>
@@ -203,5 +203,5 @@
                 <sphere radius="${caster_wheel_radius}"/>
             </geometry>
-        </collison>
+        </collision>
         <!-- INERTIA -->
         <xacro:inertial_sphere mass="${caster_wheel_mass}" radius="${caster_wheel_radius}">
@@ -210,5 +210,5 @@
     </link>
     <!-- GAZEBO LEFT CASTER WHEEL -->
-     <gazebo reference="left_caster_wheel">
+    <gazebo reference="left_caster_wheel">
         <material>Gazebo/Black</material>
         <mu1 value="0.001"/>
@@ -219,5 +219,5 @@
         <parent link="base_link"/>
         <child link="right_caster_wheel"/>
-        <orign xyz="${caster_radius*0.75} ${chassis_radius/2} ${caster_wheel_offset_z}"/>
+        <orign xyz="${chassis_radius*0.75} ${chassis_radius/2} ${caster_wheel_offset_z}"/>
     </joint>
     <!-- REAR CASTER WHEEL LINK -->
@@ -235,5 +235,5 @@
                 <sphere radius="${caster_wheel_radius}"/>
             </geometry>
-        </collison>
+        </collision>
         <!-- INERTIA -->
         <xacro:inertial_sphere mass="${caster_wheel_mass}" radius="${caster_wheel_radius}">
@@ -242,5 +242,5 @@
     </link>
     <!-- GAZEBO RIGHT CASTER WHEEL -->
-     <gazebo reference="right_caster_wheel">
+    <gazebo reference="right_caster_wheel">
         <material>Gazebo/Black</material>
         <mu1 value="0.001"/>

Commit message: fixed chassis_joint

File: description/robot_core.xacro (robot description, xacro)
@@ -54,5 +54,5 @@
     <!-- ================================================================================== -->
     <!-- CHASSIS JOINT -->
-    <joint name="chassis_joint">
+    <joint name="chassis_joint" type="fixed">
         <parent link="base_link"/>
         <child link="chassis"/>

Commit message: error_solve

File: description/robot_core.xacro (robot description, xacro)
@@ -87,5 +87,5 @@
     <!-- ================================================================================== -->
     <!-- LEFT WHEEL JOINT -->
-    <joint name="left_wheel_joint" type="continous">
+    <joint name="left_wheel_joint" type="continuous">
         <parent link="base_link"/>
         <child link="left_wheel"/>
@@ -119,5 +119,5 @@
     <!-- ================================================================================== -->
     <!-- RIGHT WHEEL JOINT -->
-    <joint name="right_wheel_joint" type="continous">
+    <joint name="right_wheel_joint" type="continuous">
         <parent link="base_link"/>
         <child link="right_wheel"/>

Commit message: Update

File: description/robot_core.xacro (robot description, xacro)
@@ -4,6 +4,6 @@
     <!-- PARAMETERS -->
     <!-- CHASSIS PARAMETERS -->
-    <xacro:property name="chassis_radius" value="0.300"/>
-    <xacro:property name="chassis_thickness" value="0.138"/>
+    <xacro:property name="chassis_radius" value="0.250"/>
+    <xacro:property name="chassis_thickness" value="0.110"/>
     <xacro:property name="chassis_mass" value="1.0"/>
     <!-- OFFSET PARAMETERS -->
@@ -12,5 +12,5 @@
     <xacro:property name="wheel_offset_z" value="0.01"/>
     <!-- WHEELS PARAMETERS -->
-    <xacro:property name="wheel_radius" value="0.033"/>
+    <xacro:property name="wheel_radius" value="0.066"/>
     <xacro:property name="wheel_thickness" value="0.026"/>
     <xacro:property name="wheel_mass" value="0.05"/>
@@ -90,5 +90,5 @@
         <parent link="base_link"/>
         <child link="left_wheel"/>
-        <origin xyz="${chassis_radius/2} ${wheel_offset_y} 0" rpy="-${pi/2} 0 0" />
+        <origin xyz="0 ${wheel_offset_y} 0" rpy="-${pi/2} 0 0" />
         <axis xyz="0 0 1"/>
     </joint>
@@ -122,5 +122,5 @@
         <parent link="base_link"/>
         <child link="right_wheel"/>
-        <origin xyz="${chassis_radius/2} ${-wheel_offset_y} 0" rpy="${pi/2} 0 0"/>
+        <origin xyz="0 ${-wheel_offset_y} 0" rpy="${pi/2} 0 0"/>
         <axis xyz="0 0 -1"/>
     </joint>

Commit message: update

File: description/robot_core.xacro (robot description, xacro)
@@ -57,5 +57,5 @@
         <parent link="base_link"/>
         <child link="chassis"/>
-        <origin xyz="${-wheel_offset_x} 0 ${-wheel_offset_z}"/>
+        <origin xyz="0 0 ${-wheel_offset_z}"/>
     </joint>
     <!-- CHASSIS LINK -->

Commit message: Update

File: description/robot_core.xacro (robot description, xacro)
@@ -4,13 +4,14 @@
     <!-- PARAMETERS -->
     <!-- CHASSIS PARAMETERS -->
-    <xacro:property name="chassis_radius" value="0.250"/>
-    <xacro:property name="chassis_thickness" value="0.110"/>
+    <xacro:property name="chassis_length" value="0.370"/>
+    <xacro:property name="chassis_width" value="0.380"/>
+    <xacro:property name="chassis_height" value="0.140"/>
     <xacro:property name="chassis_mass" value="1.0"/>
     <!-- OFFSET PARAMETERS -->
-    <xacro:property name="wheel_offset_x" value="0.265"/>
+    <xacro:property name="wheel_offset_x" value="0.285"/>
     <xacro:property name="wheel_offset_y" value="0.148"/>
     <xacro:property name="wheel_offset_z" value="0.01"/>
     <!-- WHEELS PARAMETERS -->
-    <xacro:property name="wheel_radius" value="0.066"/>
+    <xacro:property name="wheel_radius" value="0.1"/>
     <xacro:property name="wheel_thickness" value="0.026"/>
     <xacro:property name="wheel_mass" value="0.05"/>
@@ -63,7 +64,7 @@
         <!-- VISUAL -->
         <visual>
-            <origin xyz="${chassis_radius/2} 0 ${chassis_thickness}"/>
-            <geometry>
-                <cylinder radius="${chassis_radius}" length="${chassis_thickness}"/>
+            <origin xyz="${chassis_length/2} 0 ${chassis_height}"/>
+            <geometry>
+                <box size="${chassis_length} ${chassis_width} ${chassis_height}"/>
             </geometry>
             <material name="silver"/>
@@ -71,13 +72,13 @@
         <!-- COLLISION -->
         <collision>
-            <origin xyz="${chassis_radius/2} 0 ${chassis_thickness}"/>
-            <geometry>
-                <cylinder radius="${chassis_radius}" length="${chassis_thickness}"/>
-            </geometry>
-        </collision>
-        <!-- INERTIA -->
-        <xacro:inertial_cylinder mass="${chassis_mass}" length="${chassis_thickness}" radius="${chassis_radius}">
-            <origin xyz="0 0 0" rpy="0 0 0"/>
-        </xacro:inertial_cylinder>
+            <origin xyz="${chassis_length/2} 0 ${chassis_height}"/>
+            <geometry>
+                <box size="${chassis_length} ${chassis_width} ${chassis_height}"/>
+            </geometry>
+        </collision>
+        <!-- INERTIA -->
+        <xacro:inertial_box mass="${chassis_mass}" x="${chassis_length}" y="${chassis_width}" z="${chassis_height}">
+            <origin xyz="${chassis_length/2} 0 ${chassis_height/2}" rpy="0 0 0"/>
+        </xacro:inertial_box>
     </link>
     <!-- GAZEBO CHASSIS -->
@@ -187,5 +188,5 @@
         <parent link="chassis"/>
         <child link="left_caster_wheel"/>
-        <orign xyz="${chassis_radius*0.75} ${chassis_radius/2} ${caster_wheel_offset_z}"/>
+        <orign xyz="${chassis_length*0.75} ${chassis_length/2} ${caster_wheel_offset_z}"/>
     </joint>
     <!-- LEFT CASTER WHEEL LINK -->
@@ -219,5 +220,5 @@
         <parent link="base_link"/>
         <child link="right_caster_wheel"/>
-        <orign xyz="${chassis_radius*0.75} ${chassis_radius/2} ${caster_wheel_offset_z}"/>
+        <orign xyz="${chassis_length*0.75} ${chassis_length/2} ${caster_wheel_offset_z}"/>
     </joint>
     <!-- REAR CASTER WHEEL LINK -->

Commit message: Update robot_core.xacro

File: description/robot_core.xacro (robot description, xacro)
@@ -20,5 +20,5 @@
     <xacro:property name="caster_wheel_mass" value="0.01"/>
     <!-- CASTER WHEEL OFFSET PARAMTERS -->
-    <xacro:property name="caster_wheel_offset_x" value="0.075"/>
+    <xacro:property name="caster_wheel_offset_x" value="0.1"/>
     <xacro:property name="caster_wheel_offset_z" value="${wheel_offset_z - wheel_radius + caster_wheel_radius}"/>
     <!-- ================================================================================== -->
@@ -64,5 +64,5 @@
         <!-- VISUAL -->
         <visual>
-            <origin xyz="${chassis_length/2} 0 ${chassis_height}"/>
+            <origin xyz="0 0 0.05"/>
             <geometry>
                 <box size="${chassis_length} ${chassis_width} ${chassis_height}"/>
@@ -72,5 +72,5 @@
         <!-- COLLISION -->
         <collision>
-            <origin xyz="${chassis_length/2} 0 ${chassis_height}"/>
+            <origin xyz="0 0 ${chassis_height}"/>
             <geometry>
                 <box size="${chassis_length} ${chassis_width} ${chassis_height}"/>
@@ -79,5 +79,5 @@
         <!-- INERTIA -->
         <xacro:inertial_box mass="${chassis_mass}" x="${chassis_length}" y="${chassis_width}" z="${chassis_height}">
-            <origin xyz="${chassis_length/2} 0 ${chassis_height/2}" rpy="0 0 0"/>
+            <origin xyz="0 0 ${chassis_height/2}" rpy="0 0 0"/>
         </xacro:inertial_box>
     </link>
@@ -154,7 +154,7 @@
     <!-- REAR CASTER WHEEL JOINT -->
     <joint name="rear_caster_wheel_joint" type="fixed">
-        <parent link="chassis"/>
+        <parent link="base_link"/>
         <child link="rear_caster_wheel"/>
-        <orign xyz="${caster_wheel_offset_x} 0 ${caster_wheel_offset_z}"/>
+        <orign xyz="0.300 0.260 ${caster_wheel_offset_z}"/>
     </joint>
     <!-- REAR CASTER WHEEL LINK -->
@@ -220,5 +220,5 @@
         <parent link="base_link"/>
         <child link="right_caster_wheel"/>
-        <orign xyz="${chassis_length*0.75} ${chassis_length/2} ${caster_wheel_offset_z}"/>
+        <orign xyz="${chassis_length} ${chassis_width} ${caster_wheel_offset_z}"/>
     </joint>
     <!-- REAR CASTER WHEEL LINK -->

Commit message: URDF Error Solved

File: description/robot_core.xacro (robot description, xacro)
@@ -20,5 +20,6 @@
     <xacro:property name="caster_wheel_mass" value="0.01"/>
     <!-- CASTER WHEEL OFFSET PARAMTERS -->
-    <xacro:property name="caster_wheel_offset_x" value="0.1"/>
+    <xacro:property name="caster_wheel_offset_x" value="0.13"/>
+    <xacro:property name="caster_wheel_offset_y" value="0.11"/>
     <xacro:property name="caster_wheel_offset_z" value="${wheel_offset_z - wheel_radius + caster_wheel_radius}"/>
     <!-- ================================================================================== -->
@@ -156,5 +157,5 @@
         <parent link="base_link"/>
         <child link="rear_caster_wheel"/>
-        <orign xyz="0.300 0.260 ${caster_wheel_offset_z}"/>
+        <origin xyz="${-caster_wheel_offset_x} 0 ${caster_wheel_offset_z}"/>
     </joint>
     <!-- REAR CASTER WHEEL LINK -->
@@ -188,5 +189,5 @@
         <parent link="chassis"/>
         <child link="left_caster_wheel"/>
-        <orign xyz="${chassis_length*0.75} ${chassis_length/2} ${caster_wheel_offset_z}"/>
+        <origin xyz="0.15 ${caster_wheel_offset_y} ${caster_wheel_offset_z}"/>
     </joint>
     <!-- LEFT CASTER WHEEL LINK -->
@@ -220,5 +221,5 @@
         <parent link="base_link"/>
         <child link="right_caster_wheel"/>
-        <orign xyz="${chassis_length} ${chassis_width} ${caster_wheel_offset_z}"/>
+        <origin xyz="0.15 ${-caster_wheel_offset_y} ${caster_wheel_offset_z}"/>
     </joint>
     <!-- REAR CASTER WHEEL LINK -->

Commit message: wheel_offset_z Update

File: description/robot_core.xacro (robot description, xacro)
@@ -11,5 +11,5 @@
     <xacro:property name="wheel_offset_x" value="0.285"/>
     <xacro:property name="wheel_offset_y" value="0.148"/>
-    <xacro:property name="wheel_offset_z" value="0.01"/>
+    <xacro:property name="wheel_offset_z" value="0.08"/>
     <!-- WHEELS PARAMETERS -->
     <xacro:property name="wheel_radius" value="0.1"/>

Commit message: wheel_offset_z Solved

File: description/robot_core.xacro (robot description, xacro)
@@ -11,5 +11,5 @@
     <xacro:property name="wheel_offset_x" value="0.285"/>
     <xacro:property name="wheel_offset_y" value="0.148"/>
-    <xacro:property name="wheel_offset_z" value="0.08"/>
+    <xacro:property name="wheel_offset_z" value="0.005"/>
     <!-- WHEELS PARAMETERS -->
     <xacro:property name="wheel_radius" value="0.1"/>

Commit message: Wheel_offset reduced

File: description/robot_core.xacro (robot description, xacro)
@@ -92,5 +92,5 @@
         <parent link="base_link"/>
         <child link="left_wheel"/>
-        <origin xyz="0 ${wheel_offset_y} 0" rpy="-${pi/2} 0 0" />
+        <origin xyz="-0.01 ${wheel_offset_y} 0" rpy="-${pi/2} 0 0" />
         <axis xyz="0 0 1"/>
     </joint>
@@ -124,5 +124,5 @@
         <parent link="base_link"/>
         <child link="right_wheel"/>
-        <origin xyz="0 ${-wheel_offset_y} 0" rpy="${pi/2} 0 0"/>
+        <origin xyz="-0.01 ${-wheel_offset_y} 0" rpy="${pi/2} 0 0"/>
         <axis xyz="0 0 -1"/>
     </joint>

Commit message: Update base footprint

File: description/robot_core.xacro (robot description, xacro)
@@ -50,7 +50,15 @@
     </material>
     <!-- ================================================================================== -->
-    <!-- BASE FOOTPRINT -->
     <!-- BASE LINK -->
     <link name="base_link">
+    </link>
+    <!-- BASE FOOTPRINT JOINT -->
+    <joint name="base_footprint_joint" type="fixed">
+        <parent link="base_link"/>
+        <child link="base_footprint"/>
+        <origin xyz="0 0 0" rpy="0 0 0"/>
+    </joint>
+    <!-- BASE FOOTPRINT LINK -->
+    <link name="base_footprint">
     </link>
     <!-- ================================================================================== -->
