Commit message: Extra 3 TOF Integration [urdf, ros2_control, curio_hardware]

File: description/ros2_control.xacro (robot description, xacro)
@@ -8,5 +8,5 @@
             <param name="device">/dev/ttyACM0</param>
             <param name="baud_rate">57600</param>
-            <param name="timeout_ms">1000</param>
+            <param name="timeout_ms">2000</param>
             <param name="loop_rate">30</param>
             <param name="enc_counts_per_rev">752</param>

File: description/tof.xacro (robot description, xacro)
@@ -70,4 +70,69 @@
         <origin xyz="0.192 -0.148 0.06" rpy="0 0 -0.523599"/>
     </joint>
+<!-- ======================================================================== -->
+    <link name="tof_4">
+        <visual>
+            <geometry>
+                <cylinder radius="0.01" length="0.01"/>
+            </geometry>
+            <material name="red"/>
+        </visual>
+        <collision>
+            <geometry>
+                <cylinder radius="0.01" length="0.01"/>
+            </geometry>
+        </collision>
+        <xacro:inertial_cylinder mass="0.01" length="0.01" radius="0.01">
+            <origin xyz="0 0 0" rpy="0 0 0"/>
+        </xacro:inertial_cylinder>
+    </link>
+    <joint name="tof_joint_4" type="fixed">
+        <parent link="chassis"/>
+        <child link="tof_4"/>
+        <origin xyz="0.192 0.120 0.580" rpy="0 0 0"/>
+    </joint>
+    <link name="tof_5">
+        <visual>
+            <geometry>
+                <cylinder radius="0.01" length="0.01"/>
+            </geometry>
+            <material name="red"/>
+        </visual>
+        <collision>
+            <geometry>
+                <cylinder radius="0.01" length="0.01"/>
+            </geometry>
+        </collision>
+        <xacro:inertial_cylinder mass="0.01" length="0.01" radius="0.01">
+            <origin xyz="0 0 0" rpy="0 0 0"/>
+        </xacro:inertial_cylinder>
+    </link>
+    <joint name="tof_joint_5" type="fixed">
+        <parent link="chassis"/>
+        <child link="tof_5"/>
+        <origin xyz="0.192 0.0 0.560" rpy="0 0 0"/>
+    </joint>
+    <link name="tof_6">
+        <visual>
+            <geometry>
+                <cylinder radius="0.01" length="0.01"/>
+            </geometry>
+            <material name="red"/>
+        </visual>
+        <collision>
+            <geometry>
+                <cylinder radius="0.01" length="0.01"/>
+            </geometry>
+        </collision>
+        <xacro:inertial_cylinder mass="0.01" length="0.01" radius="0.01">
+            <origin xyz="0 0 0" rpy="0 0 0"/>
+        </xacro:inertial_cylinder>
+    </link>
+    <joint name="tof_joint_6" type="fixed">
+        <parent link="chassis"/>
+        <child link="tof_6"/>
+        <origin xyz="0.192 -0.120 0.580" rpy="0 0 0"/>
+    </joint>
+<!-- ==================================================== -->
     <gazebo reference="tof">
         <material>Gazebo/Red</material>
@@ -82,31 +147,19 @@
                         <samples>5</samples>
                         <resolution>1.00</resolution>
-                        <min_angle>-0.18</min_angle>
-                        <max_angle>0.18</max_angle>
-                    </horizontal>
-                    <vertical>
-                        <samples>5</samples>
-                        <resolution>1.00</resolution>
-                        <min_angle>-0.01</min_angle>
-                        <max_angle>0.01</max_angle>
-                    </vertical>
-              </scan>
-              <range>
-                    <min>0.3</min>
-                    <max>12</max>
-                    <resolution>0.01</resolution>
-              </range>
-              <noise>
-                    <type>gaussian</type>
-                    <mean>0.0</mean>
-                    <stddev>0.01</stddev>
-              </noise>
-            </ray>
-            <plugin name="bytes_laserscan" filename="libgazebo_ros_ray_sensor.so">
-              <ros>
-                  <namespace>distance</namespace>
-                <remapping>~/out:=range</remapping>
-              </ros>
-              <output_type>sensor_msgs/Range</output_type>
+                        <min_angle>-0.01</min_angle>
+                        <max_angle>0.01</max_angle>
+                    </horizontal>
+              </scan>
+              <range>
+                    <min>0.04</min>
+                    <max>12</max>
+              </range>
+            </ray>
+            <plugin name="laser_controller" filename="libgazebo_ros_ray_sensor.so">
+              <ros>
+                  <namespace>distance</namespace>
+                  <remapping>~/out:=range</remapping>
+              </ros>
+              <output_type>sensor_msgs/LaserScan</output_type>
               <frame_name>tof</frame_name>
             </plugin>
@@ -125,31 +178,19 @@
                         <samples>5</samples>
                         <resolution>1.00</resolution>
-                        <min_angle>-0.18</min_angle>
-                        <max_angle>0.18</max_angle>
-                    </horizontal>
-                    <vertical>
-                        <samples>5</samples>
-                        <resolution>1.00</resolution>
-                        <min_angle>-0.01</min_angle>
-                        <max_angle>0.01</max_angle>
-                    </vertical>
-              </scan>
-              <range>
-                    <min>0.3</min>
-                    <max>12</max>
-                    <resolution>0.01</resolution>
-              </range>
-              <noise>
-                    <type>gaussian</type>
-                    <mean>0.0</mean>
-                    <stddev>0.01</stddev>
-              </noise>
-            </ray>
-            <plugin name="bytes_laserscan" filename="libgazebo_ros_ray_sensor.so">
-              <ros>
-                  <namespace>distance</namespace>
-                <remapping>~/out:=range</remapping>
-              </ros>
-              <output_type>sensor_msgs/Range</output_type>
+                        <min_angle>-0.01</min_angle>
+                        <max_angle>0.01</max_angle>
+                    </horizontal>
+              </scan>
+              <range>
+                    <min>0.04</min>
+                    <max>12</max>
+              </range>
+            </ray>
+            <plugin name="laser_controller" filename="libgazebo_ros_ray_sensor.so">
+              <ros>
+                  <namespace>distance</namespace>
+                  <remapping>~/out:=range_1</remapping>
+              </ros>
+              <output_type>sensor_msgs/LaserScan</output_type>
               <frame_name>tof_1</frame_name>
             </plugin>
@@ -168,34 +209,115 @@
                         <samples>5</samples>
                         <resolution>1.00</resolution>
-                        <min_angle>-0.18</min_angle>
-                        <max_angle>0.18</max_angle>
-                    </horizontal>
-                    <vertical>
-                        <samples>5</samples>
-                        <resolution>1.00</resolution>
-                        <min_angle>-0.01</min_angle>
-                        <max_angle>0.01</max_angle>
-                    </vertical>
-              </scan>
-              <range>
-                    <min>0.3</min>
-                    <max>12</max>
-                    <resolution>0.01</resolution>
-              </range>
-              <noise>
-                    <type>gaussian</type>
-                    <mean>0.0</mean>
-                    <stddev>0.01</stddev>
-              </noise>
-            </ray>
-            <plugin name="bytes_laserscan" filename="libgazebo_ros_ray_sensor.so">
-              <ros>
-                  <namespace>distance</namespace>
-                <remapping>~/out:=range</remapping>
-              </ros>
-              <output_type>sensor_msgs/Range</output_type>
+                        <min_angle>-0.01</min_angle>
+                        <max_angle>0.01</max_angle>
+                    </horizontal>
+              </scan>
+              <range>
+                    <min>0.04</min>
+                    <max>12</max>
+              </range>
+            </ray>
+            <plugin name="laser_controller" filename="libgazebo_ros_ray_sensor.so">
+              <ros>
+                  <namespace>distance</namespace>
+                <remapping>~/out:=range_2</remapping>
+              </ros>
+              <output_type>sensor_msgs/LaserScan</output_type>
               <frame_name>tof_2</frame_name>
             </plugin>
         </sensor>
     </gazebo>
+    <gazebo reference="tof_4">
+        <material>Gazebo/Red</material>
+        <sensor name="tof_4" type="ray">
+            <always_on>true</always_on>
+            <visualize>true</visualize>
+            <pose>0.192 0 0.06 0 0 0</pose>
+            <update_rate>10</update_rate>
+            <ray>
+              <scan>
+                    <horizontal>
+                        <samples>5</samples>
+                        <resolution>1.00</resolution>
+                        <min_angle>-0.01</min_angle>
+                        <max_angle>0.01</max_angle>
+                    </horizontal>
+              </scan>
+              <range>
+                    <min>0.04</min>
+                    <max>12</max>
+              </range>
+            </ray>
+            <plugin name="laser_controller" filename="libgazebo_ros_ray_sensor.so">
+              <ros>
+                  <namespace>distance</namespace>
+                <remapping>~/out:=range_4</remapping>
+              </ros>
+              <output_type>sensor_msgs/LaserScan</output_type>
+              <frame_name>tof_4</frame_name>
+            </plugin>
+        </sensor>
+    </gazebo>
+    <gazebo reference="tof_5">
+        <material>Gazebo/Red</material>
+        <sensor name="tof_5" type="ray">
+            <always_on>true</always_on>
+            <visualize>true</visualize>
+            <pose>0.192 0 0.06 0 0 0</pose>
+            <update_rate>10</update_rate>
+            <ray>
+              <scan>
+                    <horizontal>
+                        <samples>5</samples>
+                        <resolution>1.00</resolution>
+                        <min_angle>-0.01</min_angle>
+                        <max_angle>0.01</max_angle>
+                    </horizontal>
+              </scan>
+              <range>
+                    <min>0.04</min>
+                    <max>12</max>
+              </range>
+            </ray>
+            <plugin name="laser_controller" filename="libgazebo_ros_ray_sensor.so">
+              <ros>
+                  <namespace>distance</namespace>
+                <remapping>~/out:=range_5</remapping>
+              </ros>
+              <output_type>sensor_msgs/LaserScan</output_type>
+              <frame_name>tof_5</frame_name>
+            </plugin>
+        </sensor>
+    </gazebo>
+    <gazebo reference="tof_6">
+        <material>Gazebo/Red</material>
+        <sensor name="tof_6" type="ray">
+            <always_on>true</always_on>
+            <visualize>true</visualize>
+            <pose>0.192 0 0.06 0 0 0</pose>
+            <update_rate>10</update_rate>
+            <ray>
+              <scan>
+                    <horizontal>
+                        <samples>5</samples>
+                        <resolution>1.00</resolution>
+                        <min_angle>-0.01</min_angle>
+                        <max_angle>0.01</max_angle>
+                    </horizontal>
+              </scan>
+              <range>
+                    <min>0.04</min>
+                    <max>12</max>
+              </range>
+            </ray>
+            <plugin name="laser_controller" filename="libgazebo_ros_ray_sensor.so">
+              <ros>
+                  <namespace>distance</namespace>
+                <remapping>~/out:=range_6</remapping>
+              </ros>
+              <output_type>sensor_msgs/LaserScan</output_type>
+              <frame_name>tof_6</frame_name>
+            </plugin>
+        </sensor>
+    </gazebo>
 </robot>

Commit message: Update TOF_INTEGRATION with Nav2_params Update

File: description/ros2_control.xacro (robot description, xacro)
@@ -9,5 +9,5 @@
             <param name="baud_rate">57600</param>
             <param name="timeout_ms">2000</param>
-            <param name="loop_rate">30</param>
+            <param name="loop_rate">50</param>
             <param name="enc_counts_per_rev">752</param>
         </hardware>
@@ -26,4 +26,9 @@
             <state_interface name="Sensor1"/>
             <state_interface name="Sensor2"/>
+            <state_interface name="Sensor4"/>
+            <state_interface name="Sensor5"/>
+            <state_interface name="Sensor6"/>
+            <state_interface name="Sensor7"/>
+            <state_interface name="Sensor8"/>
             <param name="frame_id">tof</param>
         </sensor>

File: description/tof.xacro (robot description, xacro)
@@ -47,5 +47,5 @@
         <parent link="chassis"/>
         <child link="tof_1"/>
-        <origin xyz="0.192 0.148 0.06" rpy="0 0 0.523599"/>
+        <origin xyz="0.192 -0.200 0.06" rpy="0 0 -0.523599"/>
     </joint>
     <link name="tof_2">
@@ -68,7 +68,7 @@
         <parent link="chassis"/>
         <child link="tof_2"/>
-        <origin xyz="0.192 -0.148 0.06" rpy="0 0 -0.523599"/>
-    </joint>
-<!-- ======================================================================== -->
+        <origin xyz="0.192 0.200 0.06" rpy="0 0 0.523599"/>
+    </joint>
+<!-- ============================================UPPER TOF SENSOR==================================================== -->
     <link name="tof_4">
         <visual>
@@ -134,5 +134,48 @@
         <origin xyz="0.192 -0.120 0.580" rpy="0 0 0"/>
     </joint>
-<!-- ==================================================== -->
+    <!-- ======================================LOWER DOWN SENSOR=============================================== -->
+    <link name="tof_7">
+        <visual>
+            <geometry>
+                <cylinder radius="0.01" length="0.01"/>
+            </geometry>
+            <material name="red"/>
+        </visual>
+        <collision>
+            <geometry>
+                <cylinder radius="0.01" length="0.01"/>
+            </geometry>
+        </collision>
+        <xacro:inertial_cylinder mass="0.01" length="0.01" radius="0.01">
+            <origin xyz="0 0 0" rpy="0 0 0"/>
+        </xacro:inertial_cylinder>
+    </link>
+    <joint name="tof_joint_7" type="fixed">
+        <parent link="chassis"/>
+        <child link="tof_7"/>
+        <origin xyz="0.192 -0.200 0.06" rpy="0 0 -0.523599"/>
+    </joint>
+    <link name="tof_8">
+        <visual>
+            <geometry>
+                <cylinder radius="0.01" length="0.01"/>
+            </geometry>
+            <material name="red"/>
+        </visual>
+        <collision>
+            <geometry>
+                <cylinder radius="0.01" length="0.01"/>
+            </geometry>
+        </collision>
+        <xacro:inertial_cylinder mass="0.01" length="0.01" radius="0.01">
+            <origin xyz="0 0 0" rpy="0 0 0"/>
+        </xacro:inertial_cylinder>
+    </link>
+    <joint name="tof_joint_8" type="fixed">
+        <parent link="chassis"/>
+        <child link="tof_8"/>
+        <origin xyz="0.192 0.200 0.06" rpy="0 0 0.523599"/>
+    </joint>
+<!-- =================================================================GAZEBO===================================================== -->
     <gazebo reference="tof">
         <material>Gazebo/Red</material>
@@ -193,5 +236,5 @@
               </ros>
               <output_type>sensor_msgs/LaserScan</output_type>
-              <frame_name>tof_1</frame_name>
+              <frame_name>tof</frame_name>
             </plugin>
         </sensor>
@@ -224,5 +267,5 @@
               </ros>
               <output_type>sensor_msgs/LaserScan</output_type>
-              <frame_name>tof_2</frame_name>
+              <frame_name>tof</frame_name>
             </plugin>
         </sensor>
@@ -255,5 +298,5 @@
               </ros>
               <output_type>sensor_msgs/LaserScan</output_type>
-              <frame_name>tof_4</frame_name>
+              <frame_name>tof</frame_name>
             </plugin>
         </sensor>
@@ -286,5 +329,5 @@
               </ros>
               <output_type>sensor_msgs/LaserScan</output_type>
-              <frame_name>tof_5</frame_name>
+              <frame_name>tof</frame_name>
             </plugin>
         </sensor>
@@ -317,5 +360,67 @@
               </ros>
               <output_type>sensor_msgs/LaserScan</output_type>
-              <frame_name>tof_6</frame_name>
+              <frame_name>tof</frame_name>
+            </plugin>
+        </sensor>
+    </gazebo>
+    <gazebo reference="tof_7">
+        <material>Gazebo/Red</material>
+        <sensor name="tof_7" type="ray">
+            <always_on>true</always_on>
+            <visualize>true</visualize>
+            <pose>0.192 0 0.06 0 0 0</pose>
+            <update_rate>10</update_rate>
+            <ray>
+              <scan>
+                    <horizontal>
+                        <samples>5</samples>
+                        <resolution>1.00</resolution>
+                        <min_angle>-0.01</min_angle>
+                        <max_angle>0.01</max_angle>
+                    </horizontal>
+              </scan>
+              <range>
+                    <min>0.04</min>
+                    <max>12</max>
+              </range>
+            </ray>
+            <plugin name="laser_controller" filename="libgazebo_ros_ray_sensor.so">
+              <ros>
+                  <namespace>distance</namespace>
+                <remapping>~/out:=range_7</remapping>
+              </ros>
+              <output_type>sensor_msgs/LaserScan</output_type>
+              <frame_name>tof</frame_name>
+            </plugin>
+        </sensor>
+    </gazebo>
+    <gazebo reference="tof_8">
+        <material>Gazebo/Red</material>
+        <sensor name="tof_8" type="ray">
+            <always_on>true</always_on>
+            <visualize>true</visualize>
+            <pose>0.192 0 0.06 0 0 0</pose>
+            <update_rate>10</update_rate>
+            <ray>
+              <scan>
+                    <horizontal>
+                        <samples>5</samples>
+                        <resolution>1.00</resolution>
+                        <min_angle>-0.01</min_angle>
+                        <max_angle>0.01</max_angle>
+                    </horizontal>
+              </scan>
+              <range>
+                    <min>0.04</min>
+                    <max>12</max>
+              </range>
+            </ray>
+            <plugin name="laser_controller" filename="libgazebo_ros_ray_sensor.so">
+              <ros>
+                  <namespace>distance</namespace>
+                <remapping>~/out:=range_8</remapping>
+              </ros>
+              <output_type>sensor_msgs/LaserScan</output_type>
+              <frame_name>tof</frame_name>
             </plugin>
         </sensor>

Commit message: Update

File: description/ros2_control.xacro (robot description, xacro)
@@ -8,6 +8,6 @@
             <param name="device">/dev/ttyACM0</param>
             <param name="baud_rate">57600</param>
-            <param name="timeout_ms">2000</param>
-            <param name="loop_rate">45</param>
+            <param name="timeout_ms">1000</param>
+            <param name="loop_rate">30</param>
             <param name="enc_counts_per_rev">752</param>
         </hardware>
@@ -26,9 +26,9 @@
             <state_interface name="Sensor1"/>
             <state_interface name="Sensor2"/>
+            <state_interface name="Sensor7"/>
+            <state_interface name="Sensor8"/>
             <state_interface name="Sensor4"/>
             <state_interface name="Sensor5"/>
             <state_interface name="Sensor6"/>
-            <state_interface name="Sensor7"/>
-            <state_interface name="Sensor8"/>
             <param name="frame_id">tof</param>
         </sensor>

File: description/tof.xacro (robot description, xacro)
@@ -26,5 +26,5 @@
         <parent link="chassis"/>
         <child link="tof"/>
-        <origin xyz="0.192 0.0 0.16" rpy="0 0 0"/>
+        <origin xyz="0.192 0.0 0.580" rpy="0 0 0"/>
     </joint>
     <link name="tof_1">
@@ -47,5 +47,5 @@
         <parent link="chassis"/>
         <child link="tof_1"/>
-        <origin xyz="0.192 -0.200 0.16" rpy="0 0 -0.523599"/>
+        <origin xyz="0.192 -0.120 0.580" rpy="0 0 -0.523599"/>
     </joint>
     <link name="tof_2">
@@ -68,5 +68,5 @@
         <parent link="chassis"/>
         <child link="tof_2"/>
-        <origin xyz="0.192 0.200 0.16" rpy="0 0 0.523599"/>
+        <origin xyz="0.192 0.120 0.580" rpy="0 0 0.523599"/>
     </joint>
 <!-- ============================================UPPER TOF SENSOR==================================================== -->
@@ -90,5 +90,5 @@
         <parent link="chassis"/>
         <child link="tof_4"/>
-        <origin xyz="0.192 0.120 0.580" rpy="0 0 0"/>
+        <origin xyz="0.192 -0.100 0.06" rpy="0 0 0"/>
     </joint>
     <link name="tof_5">
@@ -111,5 +111,5 @@
         <parent link="chassis"/>
         <child link="tof_5"/>
-        <origin xyz="0.192 0.0 0.560" rpy="0 0 0"/>
+        <origin xyz="0.192 0.0 0.06" rpy="0 0 0"/>
     </joint>
     <link name="tof_6">
@@ -132,5 +132,5 @@
         <parent link="chassis"/>
         <child link="tof_6"/>
-        <origin xyz="0.192 -0.120 0.580" rpy="0 0 0"/>
+        <origin xyz="0.192 0.100 0.06" rpy="0 0 0"/>
     </joint>
 <!-- ======================================LOWER DOWN SENSOR=============================================== -->
@@ -154,5 +154,5 @@
         <parent link="chassis"/>
         <child link="tof_7"/>
-        <origin xyz="0.192 -0.200 0.06" rpy="0 0 -0.523599"/>
+        <origin xyz="0.172 -0.200 0.06" rpy="0 0 -${pi/2}"/>
     </joint>
     <link name="tof_8">
@@ -175,5 +175,5 @@
         <parent link="chassis"/>
         <child link="tof_8"/>
-        <origin xyz="0.192 0.200 0.06" rpy="0 0 0.523599"/>
+        <origin xyz="0.172 0.200 0.06" rpy="0 0 ${pi/2}"/>
     </joint>
 <!-- =================================================================GAZEBO===================================================== -->
